File: temp sensor.sch (KiCad schematic (older format))
At the start: 33 parts

Commit message: added several parts, associated footprints, added todo list
Signed-off-by: lokimetasmith <lokimail@gmail.com>
Parts:
- removed U?: AHT20, Package_TO_SOT_SMD:SOT-23-6, symbol ESP32-C3-MINI-1:AHT20
- removed U?: BME680, Package_LGA:Bosch_LGA-8_3x3mm_P0.8mm_ClockwisePinNumbering, symbol Sensor:BME680
- removed U?: MS5611-01BA, Package_LGA:LGA-8_3x5mm_P1.25mm, symbol Sensor_Pressure:MS5611-01BA
- added R? (x2): 27, symbol Device:R_Small_US
- added R? (x2): 15K, symbol Device:R_Small_US
- added U?: SN65220, Package_TO_SOT_SMD:SOT-23-6, symbol Power_Protection:SN65220
- added U?: LIS2DE12, Package_LGA:LGA-12_2x2mm_P0.5mm, symbol Sensor_Motion:LIS2DE12
- added U?: Si7020-A20, Package_DFN_QFN:DFN-6-1EP_3x3mm_P1mm_EP1.5x2.4mm, symbol Sensor_Humidity:Si7020-A20
Connections:
- wire segments 186 -> 211
Other:
- note added: "AHT20 pin compatable but rotated 180"
- note added: "Accelerometer"
- note added: "KXOB25-12X1F-TR\nMONOCRYS SOLAR CELL 24.5MW 690MV"
- note added: "LIS2DS12"
- note added: "M3406-ADJ\nhttps://lcsc.com/product-detail/DC-DC-Converters_M3406_C83224.html"
- note added: "MC3479"
- note added: "Removing Capacitance soil moisture measuring for now"
- note added: "pin compatable with ESP32-PICO-MINI-02"
- moved on the sheet: C?, J?, R?

Commit message: assigned designators Signed-off-by: lokimetasmith <lokimail@gmail.com>
Parts:
- C1, C2, C3, C4, C5, C6, C7, C8, C9: renamed from C?; footprint (none) -> Capacitor_SMD:C_0603_1608Metric
- D1: renamed from D?; footprint (none) -> Diode_SMD:D_0603_1608Metric
- J1: renamed from J?; footprint (none) -> Connector_PinHeader_2.54mm:PinHeader_1x02_P2.54mm_Horizontal
- J2, J3: renamed from J?; footprint (none) -> Connector_PinHeader_2.54mm:PinHeader_1x03_P2.54mm_Vertical
- J4: renamed from J?; footprint (none) -> Connector_USB:USB_C_Plug_Molex_105444
- L1, L2: renamed from L?; footprint (none) -> Inductor_SMD:L_0603_1608Metric
- R1, R10, R11, R12, R13, R2, R3, R4, R5, R6, R7, R8, R9: renamed from R?; footprint (none) -> Resistor_SMD:R_0603_1608Metric
- Y1: renamed from Y?; footprint (none) -> Oscillator:Oscillator_SMD_Abracon_ASE-4Pin_3.2x2.5mm
- gave numbers to parts that had none: 7

Commit message: updated pdf
Signed-off-by: lokimetasmith <lokimail@gmail.com>
Parts:
- removed C1: 1u, Capacitor_SMD:C_0603_1608Metric, symbol Device:C_Small
- removed C2: sensor track, Capacitor_SMD:C_0603_1608Metric, symbol Device:C_Small
- removed D1: D, Diode_SMD:D_0603_1608Metric, symbol Device:D
- removed R1: 510K, Resistor_SMD:R_0603_1608Metric, symbol Device:R_Small_US
- removed R2, R3: 10K, Resistor_SMD:R_0603_1608Metric, symbol Device:R_Small_US
Connections:
- net labels removed: CLK_OUT, Capacitance_V
- wire segments 211 -> 195
Other:
- note removed: "CLK_OUT"
Changed lines of the file:
@@
 	1    0    0    -1
 $EndComp
-$Comp
-L Device:R_Small_US R1
-U 1 1 60828B67
-P -3200 -1450
-F 0 "R1" H -3132 -1404 50  0000 L CNN
-F 1 "510K" H -3132 -1495 50  0000 L CNN
-F 2 "Resistor_SMD:R_0603_1608Metric" H -3200 -1450 50  0001 C CNN
-F 3 "~" H -3200 -1450 50  0001 C CNN
-	1    -3200 -1450
-	1    0    0    -1
-$EndComp
-$Comp
-L Device:C_Small C1
-U 1 1 60829A42
-P -2800 -1450
-F 0 "C1" H -2708 -1404 50  0000 L CNN
-F 1 "1u" H -2708 -1495 50  0000 L CNN
-F 2 "Capacitor_SMD:C_0603_1608Metric" H -2800 -1450 50  0001 C CNN
-F 3 "~" H -2800 -1450 50  0001 C CNN
-	1    -2800 -1450
-	1    0    0    -1
-$EndComp
-$Comp
-L Device:D D1
-U 1 1 6082A1A0
-P -2500 -1750
-F 0 "D1" H -2500 -1533 50  0000 C CNN
-F 1 "D" H -2500 -1624 50  0000 C CNN
-F 2 "Diode_SMD:D_0603_1608Metric" H -2500 -1750 50  0001 C CNN
-F 3 "~" H -2500 -1750 50  0001 C CNN
-	1    -2500 -1750
-	1    0    0    -1
-$EndComp
-$Comp
-L Device:R_Small_US R2
-U 1 1 6082BA46
-P -1950 -1750
-F 0 "R2" V -2155 -1750 50  0000 C CNN
-F 1 "10K" V -2064 -1750 50  0000 C CNN
-F 2 "Resistor_SMD:R_0603_1608Metric" H -1950 -1750 50  0001 C CNN
-F 3 "~" H -1950 -1750 50  0001 C CNN
-	1    -1950 -1750
-	0    1    1    0
-$EndComp
-$Comp
-L Device:C_Small C2
-U 1 1 6082CC53
-P -2200 -1450
-F 0 "C2" H -2108 -1404 50  0000 L CNN
-F 1 "sensor track" H -2108 -1495 50  0000 L CNN
-F 2 "Capacitor_SMD:C_0603_1608Metric" H -2200 -1450 50  0001 C CNN
-F 3 "~" H -2200 -1450 50  0001 C CNN
-	1    -2200 -1450
-	1    0    0    -1
-$EndComp
-Wire Wire Line
-	-2350 -1750 -2200 -1750
-Wire Wire Line
-	-2200 -1750 -2200 -1550
-Connection ~ -2200 -1750
-Wire Wire Line
-	-2200 -1750 -2050 -1750
-Wire Wire Line
-	-2800 -1550 -2800 -1750
-Wire Wire Line
-	-2800 -1750 -2650 -1750
-Wire Wire Line
-	-3200 -1550 -3200 -1750
-Wire Wire Line
-	-3200 -1750 -2800 -1750
-Connection ~ -2800 -1750
-Wire Wire Line
-	-3200 -1350 -3200 -1250
-Wire Wire Line
-	-3200 -1250 -2800 -1250
-Wire Wire Line
-	-2800 -1250 -2800 -1350
-Wire Wire Line
-	-2800 -1250 -2200 -1250
-Wire Wire Line
-	-2200 -1250 -2200 -1350
-Connection ~ -2800 -1250
-$Comp
-L power:GND #PWR01
-U 1 1 6083669F
-P -2800 -1250
-F 0 "#PWR01" H -2800 -1500 50  0001 C CNN
-F 1 "GND" H -2795 -1423 50  0000 C CNN
-F 2 "" H -2800 -1250 50  0001 C CNN
-F 3 "" H -2800 -1250 50  0001 C CNN
-	1    -2800 -1250
-	1    0    0    -1
-$EndComp
-Text Notes -1850 -1850 0    50   ~ 0
-CLK_OUT
-Text Label -1850 -1750 0    50   ~ 0
-CLK_OUT
-Text Label -3200 -1750 0    50   ~ 0
-Capacitance_V
 Wire Wire Line
 	850  6300 1150 6300
-Text Label -650 -1450 0    50   ~ 0
-CLK_OUT
-Text Label -1450 -1550 0    50   ~ 0
-Capacitance_V
-Wire Wire Line
-	-650 -1450 -300 -1450
-Wire Wire Line
-	-900 -1550 -1450 -1550
 $Comp
 L power:+3.3V #PWR020
@@
 Connection ~ 3000 5150
 $Comp
-L Device:R_Small_US R3
-U 1 1 60909F25
-P -900 -1450
-F 0 "R3" H -832 -1404 50  0000 L CNN
-F 1 "10K" H -832 -1495 50  0000 L CNN
-F 2 "Resistor_SMD:R_0603_1608Metric" H -900 -1450 50  0001 C CNN
-F 3 "~" H -900 -1450 50  0001 C CNN
-	1    -900 -1450
-	1    0    0    -1
-$EndComp
-Wire Wire Line
-	-300 -1550 -900 -1550
-$Comp
-L power:GND #PWR02
-U 1 1 609100DE
-P -900 -1250
-F 0 "#PWR02" H -900 -1500 50  0001 C CNN
-F 1 "GND" H -895 -1423 50  0000 C CNN
-F 2 "" H -900 -1250 50  0001 C CNN
-F 3 "" H -900 -1250 50  0001 C CNN
-	1    -900 -1250
-	1    0    0    -1
-$EndComp
-Wire Wire Line
-	-900 -1350 -900 -1250
-$Comp
 L power:GND #PWR05
 U 1 1 60914CC4
@@
 Wire Wire Line
 	1400 2550 2150 2550
-Connection ~ -900 -1550
 Text Label 10050 1050 2    50   ~ 0
 SCL

Commit message: minor update
Signed-off-by: lokimetasmith <lokimail@gmail.com>
Parts:
- removed U1: LIS2DE12, Package_LGA:LGA-12_2x2mm_P0.5mm, symbol Sensor_Motion:LIS2DE12
- added J?: Conn_01x04_Male, Connector_PinHeader_2.54mm:PinHeader_1x03_P2.54mm_Vertical, symbol Connector:Conn_01x04_Male
Connections:
- wire segments 195 -> 183
Changed lines of the file:
@@
-SCL
-Wire Wire Line
-	4250 2800 4450 2800
-Wire Wire Line
-	4450 3000 4250 3000
-Text Label 4250 2800 0    50   ~ 0
-SDA
-Text Label 4250 3000 0    50   ~ 0
 SCL
 Wire Wire Line
@@
 Text Label 6650 1400 2    50   ~ 0
 SCL
-$Comp
-L power:GND #PWR015
-U 1 1 60A2672E
-P 4750 3700
-F 0 "#PWR015" H 4750 3450 50  0001 C CNN
-F 1 "GND" H 4755 3527 50  0000 C CNN
-F 2 "" H 4750 3700 50  0001 C CNN
-F 3 "" H 4750 3700 50  0001 C CNN
-	1    4750 3700
-	1    0    0    -1
-$EndComp
-Wire Wire Line
-	4750 3700 4750 3550
-Wire Wire Line
-	4950 3400 4950 3550
-Wire Wire Line
-	4950 3550 4750 3550
-Connection ~ 4750 3550
-Wire Wire Line
-	4750 3550 4750 3400
 $Comp
 L power:+5V #PWR013
@@
 Wire Wire Line
 	5750 850  5750 900
-$Comp
-L power:+3.3V #PWR016
-U 1 1 60A4E060
-P 4850 2300
-F 0 "#PWR016" H 4850 2150 50  0001 C CNN
-F 1 "+3.3V" H 4865 2473 50  0000 C CNN
-F 2 "" H 4850 2300 50  0001 C CNN
-F 3 "" H 4850 2300 50  0001 C CNN
-	1    4850 2300
-	1    0    0    -1
-$EndComp
-Wire Wire Line
-	4850 2300 4850 2350
-Wire Wire Line
-	4850 2350 4950 2350
-Connection ~ 4850 2350
-Wire Wire Line
-	4850 2350 4850 2400
-Wire Wire Line
-	4950 2350 4950 2400
 $Comp
 L power:+3.3V #PWR030
@@
 Text Notes 450  -2150 0    50   ~ 0
 KXOB25-12X1F-TR\nMONOCRYS SOLAR CELL 24.5MW 690MV
-$Comp
-L Sensor_Motion:LIS2DE12 U1
-U 1 1 60DB33D8
-P 4850 2900
-F 0 "U1" H 4900 3581 50  0000 C CNN
-F 1 "LIS2DE12" H 4900 3490 50  0000 C CNN
-F 2 "Package_LGA:LGA-12_2x2mm_P0.5mm" H 5000 3450 50  0001 L CNN
-F 3 "https://www.st.com/resource/en/datasheet/lis2DE12.pdf" H 4500 2900 50  0001 C CNN
-	1    4850 2900
-	1    0    0    -1
-$EndComp
-Text Notes 4500 2000 0    50   ~ 0
+Text Notes 450  -1900 0    50   ~ 0
 MC3479
-Text Notes 4500 2100 0    50   ~ 0
+Text Notes 450  -1800 0    50   ~ 0
 LIS2DS12
-Text Notes 4500 1900 0    50   ~ 0
+Text Notes 450  -2000 0    50   ~ 0
 Accelerometer
 $Comp
@@
 Text Notes 7350 2550 0    50   ~ 0
 AHT20 pin compatable but rotated 180
-Text Label 850  2800 2    50   ~ 0
-SCL
-Text Label 850  2900 2    50   ~ 0
-SDA
-Wire Wire Line
-	650  2800 850  2800
-Wire Wire Line
-	850  2900 650  2900
 Text Label 1950 1450 0    50   ~ 0
 SCL
@@
 Text Notes 4050 7150 0    50   ~ 0
 Removing Capacitance soil moisture measuring for now
+$Comp
+L Connector:Conn_01x04_Male J?
+U 1 1 60908C06
+P 7950 4500
+F 0 "J?" H 8058 4781 50  0000 C CNN
+F 1 "Conn_01x04_Male" H 8058 4690 50  0000 C CNN
+F 2 "Connector_PinHeader_2.54mm:PinHeader_1x03_P2.54mm_Vertical" H 7950 4500 50  0001 C CNN
+F 3 "~" H 7950 4500 50  0001 C CNN
+	1    7950 4500
+	1    0    0    -1
+$EndComp
 $EndSCHEMATC

Commit message: initial layout and silk screen options
Signed-off-by: lokimetasmith <lokimail@gmail.com>
Parts:
- removed C6, C7: C_Small, Capacitor_SMD:C_0603_1608Metric, symbol Device:C_Small
- removed J?: Conn_01x04_Male, Connector_PinHeader_2.54mm:PinHeader_1x03_P2.54mm_Vertical, symbol Connector:Conn_01x04_Male
- removed U6: HDC1080, Package_SON:Texas_PWSON-N6, symbol Sensor_Humidity:HDC1080
- removed Y1: Crystal, Oscillator:Oscillator_SMD_Abracon_ASE-4Pin_3.2x2.5mm, symbol Device:Crystal
- added D1: D_TVS, Diode_SMD:D_0603_1608Metric, symbol Device:D_TVS
- added R1: 499R, Resistor_SMD:R_0603_1608Metric, symbol Device:R_Small_US
- C4: value C_Small -> 1u
- IC1: footprint ESP32C3MINI1 -> ESP32-C3-MINI-1:ESP32C3MINI1
- J1: footprint Connector_PinHeader_2.54mm:PinHeader_1x02_P2.54mm_Horizontal -> Connector_PinHeader_2.54mm:PinHeader_1x02_P2.54mm_Vertical
- J2: footprint Connector_PinHeader_2.54mm:PinHeader_1x03_P2.54mm_Vertical -> Connector_PinHeader_2.54mm:PinHeader_1x04_P2.54mm_Vertical
- J3: value Conn_01x04_Male -> Conn_01x05_Male; footprint Connector_PinHeader_2.54mm:PinHeader_1x03_P2.54mm_Vertical -> Connector_PinHeader_2.54mm:PinHeader_1x05_P2.54mm_Vertical; symbol Connector:Conn_01x04_Male -> Connector:Conn_01x05_Male
- J4: footprint Connector_USB:USB_C_Plug_Molex_105444 -> Connector_USB:USB_Micro-B_Molex-105017-0001
Connections:
- wire segments 183 -> 171
Other:
- note added: "25mil"
- note added: "HDC1080"
- moved on the sheet: C8, C9, J2, L2, R8, R9, U2
