File: temp sensor.sch (KiCad schematic (older format))
At the start: 33 parts, among them IC1 ESP32-C3-MINI-1, J1 Conn_01x02_Male, J2 Conn_01x04_Male, J3 Conn_01x05_Male, J4 USB_B_Micro, U2 TLV62569DBV, U3 BME280, U4 Si7020-A20, U5 SN65220

Commit message: bom and pcb changes, need to add a switch still.
Signed-off-by: lokimetasmith <lokimail@gmail.com>
Parts:
- removed J1: Conn_01x02_Male, Connector_PinHeader_2.54mm:PinHeader_1x02_P2.54mm_Vertical, symbol Connector:Conn_01x02_Male
- added C1: 0.1u, Capacitor_SMD:C_0603_1608Metric, symbol Device:C_Small
- added R16, R17: 10K, Resistor_SMD:R_0603_1608Metric, symbol Device:R_Small_US
- added SW1: SW_Push, symbol Switch:SW_Push
- added U1: SHTC3, Sensor_Humidity:Sensirion_DFN-4-1EP_2x2mm_P1mm_EP0.7x1.6mm, symbol Sensor_Humidity:SHTC3
- C3: footprint Capacitor_SMD:C_0603_1608Metric -> Capacitor_SMD:C_0805_2012Metric
- D1: value D_TVS -> 3.3v_TVS; footprint Diode_SMD:D_0603_1608Metric -> Diode_SMD:D_SOD-323_HandSoldering; Description (none) -> ESD Suppressors / TVS Diodes Surge Protection PP; Manufacturer_Name (none) -> Diodes Incorporated; Manufacturer_Part_Number (none) -> SD03C-7; Mouser Part Number (none) -> 621-SD03C-7; Mouser Price/Stock (none) -> $0.37/852
- D2: Description (none) -> Standard LEDs - SMD RGB Side View; Height (none) -> 1.33; Manufacturer_Name (none) -> Cree LED; Manufacturer_Part_Number (none) -> QLS6A-FKW-CNSNSF043; Mouser Part Number (none) -> 941-QLS6AFKWNSNSF043; Mouser Price/Stock (none) -> $0.40/29,835
- IC1: Mouser Price/Stock $1.90 -> $1.90/0
- R14, R15: value 10K -> 100
- R3: value 10K -> 200
- U2: Description (none) -> Switching Voltage Regulators 2.5V-5.5V input, 2-A high effi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; Manufacturer_Name (none) -> Texas Instruments; Manufacturer_Part_Number (none) -> TLV62569DBVR; Mouser Part Number (none) -> 595-TLV62569DBVR; Mouser Price/Stock (none) -> $0.60/0
- U3: Description (none) -> MEMS humidity, pressure and temperature sensor; Manufacturer_Name (none) -> Bosch Sensortec; Manufacturer_Part_Number (none) -> BME280; Mouser Part Number (none) -> 262-BME280; Mouser Price/Stock (none) -> $5.78/0
- U4: Description (none) -> Digital RH ( 4% max) & temperature sensor,; Height (none) -> 0.75; Manufacturer_Name (none) -> Silicon Labs; Manufacturer_Part_Number (none) -> SI7020-A20-GMR; Mouser Part Number (none) -> 634-SI7020-A20-GMR; Mouser Price/Stock (none) -> $2.57/0
- U5: Description (none) -> ESD Suppressors / TVS Diodes Single USB Port; Manufacturer_Name (none) -> Texas Instruments; Manufacturer_Part_Number (none) -> SN65220DBVT; Mouser Part Number (none) -> 595-SN65220DBVT; Mouser Price/Stock (none) -> $1.03/12.700
Connections:
- net +3V3: now also U3.2 (CSB), C1.1, R16.2, R17.2, U1.1 (VDD)
- net GND: now also C9.2, R10.2, R11.1, U3.5 (SDO), U5.2 (GND), U5.5 (GND), C1.2, SW1.1, U1.4 (VSS)
- net SCL: now also R17.1, U1.2 (SCL)
- net SDA: now also R16.1, U1.3 (SDA)
- net D-: now reaches J4.2 (D-), R11.2, R13.1, U5.4 (B)
- net D+: now reaches J4.3 (D+), R10.1, R12.1, U5.6 (A)
- net at C4.2, R7.2: now also SW1.2
- net at R8.1, R9.2, U2.5 (FB): no longer C9.2
- no-connect marks 14 -> 15
Other:
- note added: "LTC3109"
- note added: "Temp/Humidity option"
- note removed: "Configure temp/humidity IO lines\n"
- moved on the sheet: D2, J3, R14, R15, R3, U3, U4
