File: temp sensor.sch (KiCad schematic (older format))
At the start: 37 parts, among them IC1 ESP32-C3-MINI-1, J2 Conn_01x04_Male, J3 Conn_01x05_Male, J4 USB_B_Micro, SW1 SW_Push, U1 SHTC3, U2 TLV62569DBV, U3 BME280, U4 Si7020-A20, U5 SN65220

Commit message: added alt parts Signed-off-by: lokimetasmith <lokimail@gmail.com>
Parts:
- IC1: Alternate Part Number 1 (none) -> ESP32-PICO-MINI-02
- U4: Alt Part Number 2 (none) -> ASAIR; Alt Part Number 3 (none) -> HDC1080; Alternate Part Number 1 (none) -> AHT20
Changed lines of the file:
@@
 F 8 "356-ESP32-C3-MINI1H4" H 3300 550 50  0001 L CNN "Mouser Part Number"
 F 9 "$1.90/0" H 3300 450 50  0001 L CNN "Mouser Price/Stock"
+F 10 "ESP32-PICO-MINI-02" H 2150 1050 50  0001 C CNN "Alternate Part Number 1"
 	1    2150 1050
 	1    0    0    -1
@@
 F 8 "$2.57/0" H 9200 1850 50  0001 C CNN "Mouser Price/Stock"
 F 9 "0.75" H 9200 1850 50  0001 C CNN "Height"
+F 10 "ASAIR" H 9200 1850 50  0001 C CNN "Alt Part Number 2"
+F 11 "HDC1080" H 9200 1850 50  0001 C CNN "Alt Part Number 3"
+F 12 "AHT20" H 9200 1850 50  0001 C CNN "Alternate Part Number 1"
 	1    9200 1850
 	1    0    0    -1

Commit message: lots of layout changes, optimized RF pathway, adjusted pinout, still working on ESP32 pinout
Signed-off-by: lokimetasmith <lokimail@gmail.com>
Parts:
- C4: value 1u -> 0.1u
- SW1: footprint (none) -> Button_Switch_SMD:SW_Push_1P1T_NO_CK_KSC6xxJ
Connections:
- wire segments 206 -> 207
Changed lines of the file:
@@
 Wire Wire Line
 	2150 1750 1900 1750
-Text Label 1850 5500 2    50   ~ 0
+Text Label 4150 7200 2    50   ~ 0
 EN
 Wire Wire Line
-	1600 5500 1850 5500
+	3900 7200 4150 7200
 $Comp
 L Device:C_Small C4
 U 1 1 609271A1
-P 1100 5600
-F 0 "C4" V 1329 5600 50  0000 C CNN
-F 1 "1u" V 1238 5600 50  0000 C CNN
-F 2 "Capacitor_SMD:C_0603_1608Metric" H 1100 5600 50  0001 C CNN
-F 3 "~" H 1100 5600 50  0001 C CNN
-	1    1100 5600
+P 3600 7200
+F 0 "C4" V 3829 7200 50  0000 C CNN
+F 1 "0.1u" V 3738 7200 50  0000 C CNN
+F 2 "Capacitor_SMD:C_0603_1608Metric" H 3600 7200 50  0001 C CNN
+F 3 "~" H 3600 7200 50  0001 C CNN
+	1    3600 7200
 	0    -1   -1   0
 $EndComp
@@
 L Device:R_Small_US R7
 U 1 1 60927BBC
-P 1500 5500
-F 0 "R7" V 1295 5500 50  0000 C CNN
-F 1 "10K" V 1386 5500 50  0000 C CNN
-F 2 "Resistor_SMD:R_0603_1608Metric" H 1500 5500 50  0001 C CNN
-F 3 "~" H 1500 5500 50  0001 C CNN
-	1    1500 5500
-	0    1    1    0
-$EndComp
-Wire Wire Line
-	1200 5600 1400 5600
-Wire Wire Line
-	1400 5600 1400 5500
-Wire Wire Line
-	1250 5100 1250 5250
-Wire Wire Line
-	1250 5250 1400 5250
-Wire Wire Line
-	1400 5250 1400 5500
-Connection ~ 1400 5500
-Wire Wire Line
-	850  5600 1000 5600
+P 3900 6600
+F 0 "R7" V 3695 6600 50  0000 C CNN
+F 1 "10K" V 3786 6600 50  0000 C CNN
+F 2 "Resistor_SMD:R_0603_1608Metric" H 3900 6600 50  0001 C CNN
+F 3 "~" H 3900 6600 50  0001 C CNN
+	1    3900 6600
+	-1   0    0    1
+$EndComp
+Wire Wire Line
+	3700 7200 3900 7200
+Wire Wire Line
+	3750 6700 3750 6850
+Wire Wire Line
+	3750 6850 3900 6850
+Wire Wire Line
+	3350 7200 3500 7200
 $Comp
 L power:GND #PWR03
 U 1 1 6094DF59
-P 850 5700
-F 0 "#PWR03" H 850 5450 50  0001 C CNN
-F 1 "GND" H 855 5527 50  0000 C CNN
-F 2 "" H 850 5700 50  0001 C CNN
-F 3 "" H 850 5700 50  0001 C CNN
-	1    850  5700
-	1    0    0    -1
-$EndComp
-Wire Wire Line
-	850  5600 850  5700
-Connection ~ 850  5600
+P 3350 7300
+F 0 "#PWR03" H 3350 7050 50  0001 C CNN
+F 1 "GND" H 3355 7127 50  0000 C CNN
+F 2 "" H 3350 7300 50  0001 C CNN
+F 3 "" H 3350 7300 50  0001 C CNN
+	1    3350 7300
+	1    0    0    -1
+$EndComp
+Wire Wire Line
+	3350 7200 3350 7300
+Connection ~ 3350 7200
 $Comp
 L Device:L_Core_Ferrite_Small L1
@@
 $EndComp
 Connection ~ 5950 4200
-Text Notes 3650 6000 0    50   ~ 0
+Text Notes -2500 200  0    50   ~ 0
 ToDo:\n\n
-Text Notes 3650 6050 0    50   ~ 0
+Text Notes -2500 250  0    50   ~ 0
 Adjust switching power supply resistor adjust values
-Text Notes 3650 6350 0    50   ~ 0
+Text Notes -2500 550  0    50   ~ 0
 Figure out boot pulldown resistors
 Text Notes 350  -1500 0    50   ~ 0
 check out soil moisture sensor circuit\n
-Text Notes 3650 6650 0    50   ~ 0
+Text Notes -2500 850  0    50   ~ 0
 Figure out GPIO and which are actually needed
-Text Notes 3650 6800 0    50   ~ 0
+Text Notes -2500 1000 0    50   ~ 0
 Prototype USB interface, confirm it works
 $Comp
@@
 L Switch:SW_Push SW1
 U 1 1 60AB27C5
-P 1050 5100
-F 0 "SW1" H 1050 5385 50  0000 C CNN
-F 1 "SW_Push" H 1050 5294 50  0000 C CNN
-F 2 "" H 1050 5300 50  0001 C CNN
-F 3 "~" H 1050 5300 50  0001 C CNN
-	1    1050 5100
-	1    0    0    -1
-$EndComp
-Wire Wire Line
-	850  5100 850  5600
+P 3550 6700
+F 0 "SW1" H 3550 6985 50  0000 C CNN
+F 1 "SW_Push" H 3550 6894 50  0000 C CNN
+F 2 "Button_Switch_SMD:SW_Push_1P1T_NO_CK_KSC6xxJ" H 3550 6900 50  0001 C CNN
+F 3 "https://www.mouser.com/datasheet/2/60/ksc3-1841668.pdf" H 3550 6900 50  0001 C CNN
+	1    3550 6700
+	1    0    0    -1
+$EndComp
+Wire Wire Line
+	3350 6700 3350 7200
 $Comp
 L Device:C_Small C1
@@
 Text Notes 1250 -2000 0    50   ~ 0
 LTC3109
+Wire Wire Line
+	3900 6850 3900 7200
+Connection ~ 3900 7200
+Wire Wire Line
+	3900 6700 3900 6850
+Connection ~ 3900 6850
+$Comp
+L power:+3.3V #PWR?
+U 1 1 609EE85F
+P 3900 6400
+F 0 "#PWR?" H 3900 6250 50  0001 C CNN
+F 1 "+3.3V" H 3915 6573 50  0000 C CNN
+F 2 "" H 3900 6400 50  0001 C CNN
+F 3 "" H 3900 6400 50  0001 C CNN
+	1    3900 6400
+	1    0    0    -1
+$EndComp
+Wire Wire Line
+	3900 6400 3900 6500
 $EndSCHEMATC

Commit message: updated schematic for updated parts
Signed-off-by: lokimetasmith <lokimail@gmail.com>
Parts:
- removed R4, R5, R6: 10K, Resistor_SMD:R_0603_1608Metric, symbol Device:R_Small_US
- added C2: 0.1u, Capacitor_SMD:C_0603_1608Metric, symbol Device:C_Small
- added R18: 2.2K, Resistor_SMD:R_0603_1608Metric, symbol Device:R_Small_US
- U1: symbol Sensor_Humidity:SHTC3 -> ESP32-C3-MINI-1:SHTC1
Connections:
- net labels added: io8
- wire segments 207 -> 211
Other:
- note added: "Set the module to UART Download mode by pulling IO0 (pulled up by default) and IO2 (pulled down by\ndefault) low. The chip IOs are pulled down internally by default."
- moved on the sheet: L1

Commit message: updated bom
Signed-off-by: lokimetasmith <lokimail@gmail.com>
Parts:
- C1, C2, C4, C5: Description (none) -> Multilayer Ceramic Capacitors MLCC - SMD/SMT 0603 16VDC 0.1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; Height (none) -> 0.9; Manufacturer_Name (none) -> Taiyo Yuden; Manufacturer_Part_Number (none) -> EMK107B7104KAHT; Mouser Part Number (none) -> 963-EMK107B7104KAHT; Mouser Price/Stock (none) -> $0.10/110000
- C3, C9: Description (none) -> Multilayer Ceramic Capacitors MLCC - SMD/SMT 0805 10VDC 10u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; Manufacturer_Name (none) -> Taiyo Yuden; Manufacturer_Part_Number (none) -> LMK212ABJ106MG-T; Mouser Part Number (none) -> 963-LMK212ABJ106MG-T; Mouser Price/Stock (none) -> $0.13/104348
- C8: Description (none) -> Multilayer Ceramic Capacitors MLCC - SMD/SMT 0603 6.3VDC 4.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; Manufacturer_Name (none) -> Taiyo Yuden; Manufacturer_Part_Number (none) -> JMK107C6475KA-T; Mouser Part Number (none) -> 963-JMK107C6475KA-T; Mouser Price/Stock (none) -> $0.16/1200
- J4: Description (none) -> USB Connectors MICRO USB B RECPT BTTM MNT SMT TH TABS; Manufacturer_Name (none) -> Molex; Manufacturer_Part_Number (none) -> 105017-0001; Mouser Part Number (none) -> 538-105017-0001; Mouser Price/Stock (none) -> $0.88/15,819
- L1: Description (none) -> Ferrite Beads 100ohms 2A 40mOhms 0603 Ferrite Chip; Manufacturer_Name (none) -> TDK; Manufacturer_Part_Number (none) -> MPZ1608Y101BTA00; Mouser Part Number (none) -> 810-MPZ1608Y101BTA00
- L2: Description (none) -> Fixed Inductors 4040 2.2uH 79mOhms +/-20%Tol 2.8A HiCur; Height (none) -> 2; Manufacturer_Name (none) -> Taiyo Yuden; Manufacturer_Part_Number (none) -> MDMK4040T2R2MM; Mouser Part Number (none) -> 963-MDMK4040T2R2MM; Mouser Price/Stock (none) -> $0.78/678
- R1, R2: Description (none) -> Thick Film Resistors - SMD 499 ohm 1%; Manufacturer_Name (none) -> Bourns; Manufacturer_Part_Number (none) -> CR0603-FX-4990ELF; Mouser Part Number (none) -> 652-CR0603FX-4990ELF; Mouser Price/Stock (none) -> $0.10/19000
- R10, R11: Description (none) -> Thick Film Resistors - SMD 15 kOhms 100-200 mW 0603 1%; Manufacturer_Name (none) -> Yageo; Manufacturer_Part_Number (none) -> RC0603FR-1315KL; Mouser Part Number (none) -> 603-RC0603FR-1315KL; Mouser Price/Stock (none) -> $0.10/78000
- R12, R13: Description (none) -> Thick Film Resistors - SMD 1/8W 27 OHM 5%; Manufacturer_Name (none) -> KOA Speer; Manufacturer_Part_Number (none) -> RK73B1JTTDD270J; Mouser Part Number (none) -> 660-RK73B1JTTDD270J; Mouser Price/Stock (none) -> $0.10/100000
- R14, R15: Description (none) -> Thick Film Resistors - SMD 100 Ohms 100 mW 0603 5%; Manufacturer_Name (none) -> Yageo; Manufacturer_Part_Number (none) -> RC0603JR-07100RL; Mouser Part Number (none) -> 603-RC0603JR-07100RL; Mouser Price/Stock (none) -> $0.10/2,633,578
- R16, R17, R7: Description (none) -> Thick Film Resistors - SMD 10 kOhms 100 mW 0603 5%; Manufacturer_Name (none) -> Yageo; Manufacturer_Part_Number (none) -> ESR03EZPJ103; Mouser Part Number (none) -> 755-ESR03EZPJ103; Mouser Price/Stock (none) -> $0.10/256000
- R18: Description (none) -> Thick Film Resistors - SMD 0603 2.2KOHMS 5% 1/10WATT; Manufacturer_Name (none) -> Bourns; Manufacturer_Part_Number (none) -> CR0603-JW-222ELF; Mouser Part Number (none) -> 652-CR0603-JW-222ELF; Mouser Price/Stock (none) -> $0.10/375000
- R3: Description (none) -> Thick Film Resistors - SMD 200 OHM 1%; Manufacturer_Name (none) -> Bourns; Manufacturer_Part_Number (none) -> CR0603-FX-2000ELF; Mouser Part Number (none) -> 652-CR0603-FX2000ELF; Mouser Price/Stock (none) -> $0.10/78000
- R8: value 470k -> 680k; Description (none) -> Thick Film Resistors - SMD 680 kOhms 100-200 mW 0603 1%; Manufacturer_Name (none) -> Yageo; Manufacturer_Part_Number (none) -> RC0603FR-13680KL; Mouser Part Number (none) -> 603-RC0603FR-13680KL; Mouser Price/Stock (none) -> $0.10/100000
- R9: value 120K -> 150K; Description (none) -> Thick Film Resistors - SMD 150 kOhms 100mW 0603 1%; Manufacturer_Name (none) -> Yageo; Manufacturer_Part_Number (none) -> RC0603FR-07150KL; Mouser Part Number (none) -> 603-RC0603FR-07150KL; Mouser Price/Stock (none) -> $0.10/100000
- SW1: Description (none) -> Tactile Switches 0.3mA 24VAC, 1.60N 3.5mmH, J lead, IP67; Manufacturer_Name (none) -> C&K; Manufacturer_Part_Number (none) -> KSC2TE01JLFS; Mouser Part Number (none) -> 611-KSC2TE01JLFS; Mouser Price/Stock (none) -> $0.39/10000
- U2: Alternate Part Number 1 (none) -> MP2128DT-LF-Z; Height (none) -> b2.9/s3.5
Other:
- note added: "USB Micro B might need to be IP rated"
- note removed: "Adjust switching power supply resistor adjust values"

Commit message: exported gerbers, initial board spin
Signed-off-by: lokimetasmith <lokimail@gmail.com>
Parts:
- C1, C2, C3, C4, C5, C8, C9: symbol Device:C_Small -> temp-sensor-rescue:C_Small-Device
- D1: symbol Device:D_TVS -> temp-sensor-rescue:D_TVS-Device
- D2: symbol Device:LED_RGB -> temp-sensor-rescue:LED_RGB-Device
- J2: symbol Connector:Conn_01x04_Male -> temp-sensor-rescue:Conn_01x04_Male-Connector
- J3: symbol Connector:Conn_01x05_Male -> temp-sensor-rescue:Conn_01x05_Male-Connector
- J4: symbol Connector:USB_B_Micro -> temp-sensor-rescue:USB_B_Micro-Connector
- L1: symbol Device:L_Core_Ferrite_Small -> temp-sensor-rescue:L_Core_Ferrite_Small-Device
- L2: symbol Device:L -> Device:L_Core_Ferrite_Small
- R1, R10, R11, R12, R13, R14, R15, R16, R17, R18, R2, R3, R7, R8, R9: symbol Device:R_Small_US -> temp-sensor-rescue:R_Small_US-Device
- SW1: symbol Switch:SW_Push -> temp-sensor-rescue:SW_Push-Switch
- U2: symbol Regulator_Switching:TLV62569DBV -> temp-sensor-rescue:TLV62569DBV-Regulator_Switching
- U3: symbol Sensor:BME280 -> temp-sensor-rescue:BME280-Sensor
- U4: symbol Sensor_Humidity:Si7020-A20 -> temp-sensor-rescue:Si7020-A20-Sensor_Humidity
- U5: symbol Power_Protection:SN65220 -> temp-sensor-rescue:SN65220-Power_Protection

Commit message: minor cosmetic updates
Signed-off-by: lokimetasmith <lokimail@gmail.com>
Connections:
- net I35_pico: now reaches IC1.10 (NC_4)
- net IO25_pico: now reaches IC1.15 (NC_5)
- net IO27_pico: now reaches IC1.17 (NC_6)
- net IO4_pico: now reaches IC1.24 (NC_7)
- net IO8_pico: now reaches IC1.28 (NC_9)
- net IO5_pico: now reaches IC1.29 (NC_10)
- net IO19_pico: now reaches IC1.33 (NC_12)
- net IO22_pico: now reaches IC1.34 (NC_13)
- net IO21_pico: now reaches IC1.35 (NC_14)
- net I36_pico: now reaches IC1.4 (NC_1)
- net I39_pico: now reaches IC1.7 (NC_2)
- net I34_pico: now reaches IC1.9 (NC_3)
- net SCL renamed I38_pico
- net SDA renamed I37_pico
- net TCK renamed IO13_pico
- net TDI renamed IO12_pico
- net TDO renamed IO15_pico
- net TMS renamed IO14_pico
- net USB_D+ renamed IO7_pico
- net USB_D- renamed IO20_pico
- net io0 renamed IO32_pico
- net io1 renamed IO33_pico
- net io10 renamed IO26_pico
- net io8 renamed IO2_pico
- no-connect marks 15 -> 16
Other:
- moved on the sheet: R1, R2
Changed lines of the file:
@@
 NoConn ~ 3450 1250
 NoConn ~ 3450 1350
-NoConn ~ 2150 1350
+NoConn ~ 1800 1350
 NoConn ~ 2150 3750
 NoConn ~ 2150 3850
@@
 	5050 2450 4850 2450
 Connection ~ 4850 2450
-Text Label 1650 3650 0    50   ~ 0
+Text Label 1850 3650 0    50   ~ 0
 USB_D+
-Text Label 1650 3550 0    50   ~ 0
+Text Label 1850 3550 0    50   ~ 0
 USB_D-
-Wire Wire Line
-	1650 3550 2150 3550
-Wire Wire Line
-	2150 3650 1650 3650
-Text Label 1600 3950 0    50   ~ 0
+Text Label 1500 3950 0    50   ~ 0
 RTX0
-Text Label 1200 4050 0    50   ~ 0
+Text Label 1100 4050 0    50   ~ 0
 TDX0
 Wire Wire Line
-	1600 3950 1800 3950
+	1500 3950 1700 3950
 Text Label 7100 5250 2    50   ~ 0
 RTX0
@@
 Wire Wire Line
 	9800 5100 10150 5100
-Text Label 1650 3250 0    50   ~ 0
+Text Label 1700 3250 0    50   ~ 0
 Boot_Option
 Connection ~ 1150 6850
@@
 Text Notes 9150 4850 0    50   ~ 0
 ESD
-Text Notes 1750 2150 0    50   ~ 0
+Text Notes 1350 2150 0    50   ~ 0
 RTC\n
-Text Notes 1450 2650 0    50   ~ 0
+Text Notes 1200 2750 0    50   ~ 0
 JTAG\n
-Text Label 1650 2750 0    50   ~ 0
+Text Label 2000 2750 0    50   ~ 0
 TMS
-Text Label 1650 2850 0    50   ~ 0
+Text Label 2000 2850 0    50   ~ 0
 TDI
-Text Label 1650 2950 0    50   ~ 0
+Text Label 2000 2950 0    50   ~ 0
 TCK
-Text Label 1650 3050 0    50   ~ 0
+Text Label 2000 3050 0    50   ~ 0
 TDO
-Wire Wire Line
-	1650 2750 2150 2750
-Wire Wire Line
-	1650 2850 2150 2850
-Wire Wire Line
-	1650 2950 2150 2950
-Wire Wire Line
-	1650 3050 2150 3050
 Text Notes 4350 3700 0    50   ~ 0
 switching power supply\n
@@
 Text Label 2000 2250 0    50   ~ 0
 io1
-Wire Wire Line
-	2000 2150 2150 2150
-Wire Wire Line
-	2000 2250 2150 2250
 $Comp
 L temp-sensor-rescue:GND-power #PWR05
@@
 Wire Wire Line
 	9400 5100 8950 5100
-Text Notes 1900 650  0    50   ~ 0
-pin compatable with ESP32-PICO-MINI-02
 Text Notes 4350 3900 0    50   ~ 0
 M3406-ADJ\nhttps://lcsc.com/product-detail/DC-DC-Converters_M3406_C83224.html
@@
 Text Label 1950 1450 0    50   ~ 0
 SDA
-Wire Wire Line
-	2150 1550 1950 1550
-Wire Wire Line
-	1950 1450 2150 1450
 Text Notes 400  -1650 0    50   ~ 0
 Removing Capacitance soil moisture measuring for now
@@
 HDC1080
 Wire Wire Line
-	1600 4050 2150 4050
+	1500 4050 2150 4050
 Text Notes 1600 1250 0    50   ~ 0
 25mil
@@
 io1
 Wire Wire Line
-	2150 3950 2000 3950
+	2150 3950 1900 3950
 Wire Wire Line
 	8550 4300 8550 4200
@@
 Wire Wire Line
 	8950 4200 8950 4400
-Text Label 1650 2550 0    50   ~ 0
+Text Label 2000 2550 0    50   ~ 0
 io10
 Text Label 8950 4400 0    50   ~ 0
@@
 	3750 6850 3900 6850
 Wire Wire Line
-	1650 3250 2150 3250
-Wire Wire Line
-	1400 4050 1200 4050
-Wire Wire Line
-	1650 2550 2150 2550
-Text Label 1650 3150 0    50   ~ 0
+	1300 4050 1100 4050
+Text Label 2000 3150 0    50   ~ 0
 io8
-Wire Wire Line
-	2150 3150 1650 3150
 Wire Wire Line
 	7650 1800 7750 1800
@@
 	1    1150 6950
 	1    0    0    -1
-$EndComp
-$Comp
-L Device:L_Core_Ferrite_Small L2
-U 1 1 608A2A34
-P 5350 4200
-F 0 "L2" V 5169 4200 50  0000 C CNN
-F 1 "2.2uH" V 5260 4200 50  0000 C CNN
-F 2 "Inductor_SMD:L_Taiyo-Yuden_MD-4040" H 5350 4200 50  0001 C CNN
-F 3 "https://www.mouser.com/datasheet/2/396/wound09_e-1396591.pdf" H 5350 4200 50  0001 C CNN
-F 4 "Fixed Inductors 4040 2.2uH 79mOhms +/-20%Tol 2.8A HiCur" H 5350 4200 50  0001 C CNN "Description"
-F 5 "Taiyo Yuden" H 5350 4200 50  0001 C CNN "Manufacturer_Name"
-F 6 "MDMK4040T2R2MM" H 5350 4200 50  0001 C CNN "Manufacturer_Part_Number"
-F 7 "963-MDMK4040T2R2MM" H 5350 4200 50  0001 C CNN "Mouser Part Number"
-F 8 "	$0.78/678" H 5350 4200 50  0001 C CNN "Mouser Price/Stock"
-F 9 "2" H 5350 4200 50  0001 C CNN "Height"
-	1    5350 4200
-	0    -1   1    0
 $EndComp
 $Comp
@@
 L temp-sensor-rescue:R_Small_US-Device R1
 U 1 1 609ADAE9
-P 1500 4050
-F 0 "R1" V 1295 4050 50  0000 C CNN
-F 1 "499R" V 1386 4050 50  0000 C CNN
-F 2 "Resistor_SMD:R_0603_1608Metric" H 1500 4050 50  0001 C CNN
-F 3 "https://www.mouser.com/datasheet/2/54/crxxxxx-1858361.pdf" H 1500 4050 50  0001 C CNN
-F 4 "Thick Film Resistors - SMD 499 ohm 1%" H 1500 4050 50  0001 C CNN "Description"
-F 5 "Bourns" H 1500 4050 50  0001 C CNN "Manufacturer_Name"
-F 6 "CR0603-FX-4990ELF" H 1500 4050 50  0001 C CNN "Manufacturer_Part_Number"
-F 7 "652-CR0603FX-4990ELF" H 1500 4050 50  0001 C CNN "Mouser Part Number"
-F 8 "$0.10/19000" H 1500 4050 50  0001 C CNN "Mouser Price/Stock"
-	1    1500 4050
+P 1400 4050
+F 0 "R1" V 1195 4050 50  0000 C CNN
+F 1 "499R" V 1286 4050 50  0000 C CNN
+F 2 "Resistor_SMD:R_0603_1608Metric" H 1400 4050 50  0001 C CNN
+F 3 "https://www.mouser.com/datasheet/2/54/crxxxxx-1858361.pdf" H 1400 4050 50  0001 C CNN
+F 4 "Thick Film Resistors - SMD 499 ohm 1%" H 1400 4050 50  0001 C CNN "Description"
+F 5 "Bourns" H 1400 4050 50  0001 C CNN "Manufacturer_Name"
+F 6 "CR0603-FX-4990ELF" H 1400 4050 50  0001 C CNN "Manufacturer_Part_Number"
+F 7 "652-CR0603FX-4990ELF" H 1400 4050 50  0001 C CNN "Mouser Part Number"
+F 8 "$0.10/19000" H 1400 4050 50  0001 C CNN "Mouser Price/Stock"
+	1    1400 4050
 	0    1    1    0
 $EndComp
@@
 L temp-sensor-rescue:R_Small_US-Device R2
 U 1 1 6096A5B0
-P 1900 3950
-F 0 "R2" V 1695 3950 50  0000 C CNN
-F 1 "499R" V 1786 3950 50  0000 C CNN
-F 2 "Resistor_SMD:R_0603_1608Metric" H 1900 3950 50  0001 C CNN
-F 3 "https://www.mouser.com/datasheet/2/54/crxxxxx-1858361.pdf" H 1900 3950 50  0001 C CNN
-F 4 "Thick Film Resistors - SMD 499 ohm 1%" H 1900 3950 50  0001 C CNN "Description"
-F 5 "Bourns" H 1900 3950 50  0001 C CNN "Manufacturer_Name"
-F 6 "CR0603-FX-4990ELF" H 1900 3950 50  0001 C CNN "Manufacturer_Part_Number"
-F 7 "652-CR0603FX-4990ELF" H 1900 3950 50  0001 C CNN "Mouser Part Number"
-F 8 "$0.10/19000" H 1900 3950 50  0001 C CNN "Mouser Price/Stock"
-	1    1900 3950
+P 1800 3950
+F 0 "R2" V 1595 3950 50  0000 C CNN
+F 1 "499R" V 1686 3950 50  0000 C CNN
+F 2 "Resistor_SMD:R_0603_1608Metric" H 1800 3950 50  0001 C CNN
+F 3 "https://www.mouser.com/datasheet/2/54/crxxxxx-1858361.pdf" H 1800 3950 50  0001 C CNN
+F 4 "Thick Film Resistors - SMD 499 ohm 1%" H 1800 3950 50  0001 C CNN "Description"
+F 5 "Bourns" H 1800 3950 50  0001 C CNN "Manufacturer_Name"
+F 6 "CR0603-FX-4990ELF" H 1800 3950 50  0001 C CNN "Manufacturer_Part_Number"
+F 7 "652-CR0603FX-4990ELF" H 1800 3950 50  0001 C CNN "Mouser Part Number"
+F 8 "$0.10/19000" H 1800 3950 50  0001 C CNN "Mouser Price/Stock"
+	1    1800 3950
 	0    1    1    0
 $EndComp
@@
 Wire Wire Line
 	5450 4200 5600 4200
+$Comp
+L Device:L_Core_Ferrite_Small L2
+U 1 1 608A2A34
+P 5350 4200
+F 0 "L2" V 5169 4200 50  0000 C CNN
+F 1 "2.2uH" V 5260 4200 50  0000 C CNN
+F 2 "Inductor_SMD:L_Taiyo-Yuden_MD-4040" H 5350 4200 50  0001 C CNN
+F 3 "https://www.mouser.com/datasheet/2/396/wound09_e-1396591.pdf" H 5350 4200 50  0001 C CNN
+F 4 "Fixed Inductors 4040 2.2uH 79mOhms +/-20%Tol 2.8A HiCur" H 5350 4200 50  0001 C CNN "Description"
+F 5 "Taiyo Yuden" H 5350 4200 50  0001 C CNN "Manufacturer_Name"
+F 6 "MDMK4040T2R2MM" H 5350 4200 50  0001 C CNN "Manufacturer_Part_Number"
+F 7 "963-MDMK4040T2R2MM" H 5350 4200 50  0001 C CNN "Mouser Part Number"
+F 8 "	$0.78/678" H 5350 4200 50  0001 C CNN "Mouser Price/Stock"
+F 9 "2" H 5350 4200 50  0001 C CNN "Height"
+	1    5350 4200
+	0    -1   1    0
+$EndComp
+Text Label 1800 1350 0    50   ~ 0
+I36_pico
+Wire Wire Line
+	2150 1350 1800 1350
+Text Label 1600 1450 0    50   ~ 0
+I37_pico
+Text Label 1600 1550 0    50   ~ 0
+I38_pico
+Text Label 1600 1650 0    50   ~ 0
+I39_pico
+Wire Wire Line
+	1600 1450 2150 1450
+Wire Wire Line
+	1600 1550 2150 1550
+Wire Wire Line
+	1600 1650 2150 1650
+Text Label 1600 1850 0    50   ~ 0
+I34_pico
+Text Label 1600 1950 0    50   ~ 0
+I35_pico
+Wire Wire Line
+	1600 1850 2150 1850
+Wire Wire Line
+	2150 1950 1600 1950
+Text Label 1600 2150 0    50   ~ 0
+IO32_pico
+Text Label 1600 2250 0    50   ~ 0
+IO33_pico
+Wire Wire Line
+	1600 2150 2150 2150
+Wire Wire Line
+	1600 2250 2150 2250
+Text Label 1600 2450 0    50   ~ 0
+IO25_pico
+Wire Wire Line
+	1600 2450 2150 2450
+Text Label 1600 2550 0    50   ~ 0
+IO26_pico
+Text Label 1600 2650 0    50   ~ 0
+IO27_pico
+Text Label 1600 2750 0    50   ~ 0
+IO14_pico
+Text Label 1600 2850 0    50   ~ 0
+IO12_pico
+Text Label 1600 2950 0    50   ~ 0
+IO13_pico
+Text Label 1600 3050 0    50   ~ 0
+IO15_pico
+Wire Wire Line
+	1600 2550 2150 2550
+Wire Wire Line
+	1600 2650 2150 2650
+Wire Wire Line
+	1600 2750 2150 2750
+Wire Wire Line
+	1600 2850 2150 2850
+Wire Wire Line
+	1600 2950 2150 2950
+Wire Wire Line
+	1600 3050 2150 3050
+Text Label 1350 3150 0    50   ~ 0
+IO2_pico
+Text Label 1350 3250 0    50   ~ 0
+IO0_pico
+Text Label 1350 3350 0    50   ~ 0
+IO4_pico
+Wire Wire Line
+	1350 3150 2150 3150
+Wire Wire Line
+	1350 3250 2150 3250
+Wire Wire Line
+	1350 3350 2150 3350
+Text Label 1450 3550 0    50   ~ 0
+IO20_pico
+Text Label 1450 3650 0    50   ~ 0
+IO7_pico
+Text Label 1450 3750 0    50   ~ 0
+IO8_pico
+Text Label 1450 3850 0    50   ~ 0
+IO5_pico
+Wire Wire Line
+	1450 3550 2150 3550
+Wire Wire Line
+	1450 3650 2150 3650
+Wire Wire Line
+	1450 3750 2150 3750
+Wire Wire Line
+	2150 3850 1450 3850
+Text Label 3950 1150 2    50   ~ 0
+IO19_pico
+Text Label 3950 1250 2    50   ~ 0
+IO22_pico
+Text Label 3950 1350 2    50   ~ 0
+IO21_pico
+Wire Wire Line
+	3950 1150 3450 1150
+Wire Wire Line
+	3450 1250 3950 1250
+Wire Wire Line
+	3950 1350 3450 1350
+NoConn ~ 2150 3150
+$Comp
+L power:PWR_FLAG #FLG0101
+U 1 1 60C49CC8
+P 5600 4200
+F 0 "#FLG0101" H 5600 4275 50  0001 C CNN
+F 1 "PWR_FLAG" H 5600 4373 50  0000 C CNN
+F 2 "" H 5600 4200 50  0001 C CNN
+F 3 "~" H 5600 4200 50  0001 C CNN
+	1    5600 4200
+	1    0    0    -1
+$EndComp
+Text Notes 1900 650  0    50   ~ 0
+pin compatable with ESP32-PICO-MINI-02
 $EndSCHEMATC
