File: temp sensor.sch (KiCad schematic (older format))
At the start: 36 parts, among them IC1 ESP32-C3-MINI-1, J2 Conn_01x04_Male, J3 Conn_01x05_Male, J4 USB_B_Micro, SW1 SW_Push, U1 SHTC3, U2 TLV62569DBV, U3 BME280, U4 Si7020-A20, U5 SN65220

Commit message: first crack at v2
Signed-off-by: lokimetasmith <lokimail@gmail.com>
Parts:
- removed J2: Conn_01x04_Male, Connector_PinHeader_2.54mm:PinHeader_1x04_P2.54mm_Vertical, symbol temp-sensor-rescue:Conn_01x04_Male-Connector
- removed R18: 2.2K, Resistor_SMD:R_0603_1608Metric, symbol temp-sensor-rescue:R_Small_US-Device
- added J2, J5, J6: Conn_01x02_Male, Connector_PinHeader_2.54mm:PinHeader_1x02_P2.54mm_Vertical, symbol Connector:Conn_01x02_Male
- added Q1: BC847BDW1, Package_TO_SOT_SMD:SOT-363_SC-70-6, symbol Transistor_BJT:BC847BDW1
- added R4, R5, R6: 10K, Resistor_SMD:R_0603_1608Metric, symbol temp-sensor-rescue:R_Small_US-Device
- added SW2: SW_Push, Button_Switch_SMD:SW_Push_1P1T_NO_CK_KSC6xxJ, symbol temp-sensor-rescue:SW_Push-Switch
- D2: value LED_RGB -> QLS6A; symbol temp-sensor-rescue:LED_RGB-Device -> LED:QLS6A-FKW
- J3: footprint Connector_PinHeader_2.54mm:PinHeader_1x05_P2.54mm_Vertical -> Connector_PinSocket_1.00mm:PinSocket_1x06_P1.00mm_Vertical_SMD_Pin1Right
Connections:
- net +3V3: now also D2.1 (AB), D2.3 (AR), J2.1 (Pin_1), R6.2; no longer D2.4 (BA), D2.6 (RA)
- net Boot_Option: now also Q1.3 (C2), R6.1, SW2.2
- net EN: now also Q1.6 (C1)
- net GND: now also J2.2 (Pin_2), SW2.1
- net RTX0: now also J5.2 (Pin_2)
- net TDX0: now also J5.1 (Pin_1)
- net at R3.2: now also D2.2 (KB); no longer D2.1 (RK)
- net at R14.2: now also D2.6 (KR); no longer D2.2 (GK)
- net at R15.2: now also D2.4 (KR); no longer D2.3 (BK)
- new net: Q1.2 (B1), R4.2
- new net: Q1.5 (B2), R5.2
- new net DTR: J6.1 (Pin_1), Q1.4 (E2), R4.1
- new net RTS: J6.2 (Pin_2), Q1.1 (E1), R5.1
Other:
- moved on the sheet: C2, J3, R14, R15, R3
