File: temp sensor.sch (KiCad schematic (older format))
At the start: 42 parts, among them IC1 ESP32-C3-MINI-1, J2 Conn_01x02_Male, J3 Conn_01x05_Male, J4 USB_B_Micro, J5 Conn_01x02_Male, J6 Conn_01x02_Male, Q1 BC847BDW1, SW1 SW_Push, SW2 SW_Push, U1 SHTC3, U2 TLV62569DBV, U3 BME280, U4 Si7020-A20, U5 SN65220

Commit message: working on switch footprint
Signed-off-by: lokimetasmith <lokimail@gmail.com>
Parts:
- SW1, SW2: footprint Button_Switch_SMD:SW_Push_1P1T_NO_CK_KSC6xxJ -> Twig:SW_Push_1P1T-MP_NO_Horizontal_TL6340; Alt Part Number 3 (none) -> SKTDLHE010; Alternate Part Number 1 (none) -> EVP-AKE31A; Description Tactile Switches 0.3mA 24VAC, 1.60N 3.5mmH, J lead, IP67 -> Tactile Switch SPST-NO Side Actuated Surface Mount, Right A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; Manufacturer_Name C&K -> E-Switch; Manufacturer_Part_Number KSC2TE01JLFS -> TL6340AF160QG; Mouser Part Number 611-KSC2TE01JLFS -> (none); Mouser Price/Stock $0.39/10000 -> $0.48/10000
Changed lines of the file:
@@
 F 0 "SW1" H 3550 7135 50  0000 C CNN
 F 1 "SW_Push" H 3550 7044 50  0000 C CNN
-F 2 "Button_Switch_SMD:SW_Push_1P1T_NO_CK_KSC6xxJ" H 3550 7050 50  0001 C CNN
-F 3 "https://www.mouser.com/datasheet/2/60/ksc3-1841668.pdf" H 3550 7050 50  0001 C CNN
-F 4 "Tactile Switches 0.3mA 24VAC, 1.60N 3.5mmH, J lead, IP67" H 3550 6850 50  0001 C CNN "Description"
-F 5 "C&K" H 3550 6850 50  0001 C CNN "Manufacturer_Name"
-F 6 "KSC2TE01JLFS" H 3550 6850 50  0001 C CNN "Manufacturer_Part_Number"
-F 7 "611-KSC2TE01JLFS" H 3550 6850 50  0001 C CNN "Mouser Part Number"
-F 8 "$0.39/10000" H 3550 6850 50  0001 C CNN "Mouser Price/Stock"
+F 2 "Twig:SW_Push_1P1T-MP_NO_Horizontal_TL6340" H 3550 7050 50  0001 C CNN
+F 3 "https://sten-eswitch-13110800-production.s3.amazonaws.com/system/asset/product_line/data_sheet/256/TL6340.pdf" H 3550 7050 50  0001 C CNN
+F 4 "Tactile Switch SPST-NO Side Actuated Surface Mount, Right Angle" H 3550 6850 50  0001 C CNN "Description"
+F 5 "E-Switch" H 3550 6850 50  0001 C CNN "Manufacturer_Name"
+F 6 "TL6340AF160QG" H 3550 6850 50  0001 C CNN "Manufacturer_Part_Number"
+F 7 "" H 3550 6850 50  0001 C CNN "Mouser Part Number"
+F 8 "$0.48/10000" H 3550 6850 50  0001 C CNN "Mouser Price/Stock"
+F 9 "SKTDLHE010" H 3550 6850 50  0001 C CNN "Alt Part Number 3"
+F 10 "EVP-AKE31A" H 3550 6850 50  0001 C CNN "Alternate Part Number 1"
 	1    3550 6850
 	1    0    0    -1
@@
 F 0 "SW2" H 4700 7135 50  0000 C CNN
 F 1 "SW_Push" H 4700 7044 50  0000 C CNN
-F 2 "Button_Switch_SMD:SW_Push_1P1T_NO_CK_KSC6xxJ" H 4700 7050 50  0001 C CNN
-F 3 "https://www.mouser.com/datasheet/2/60/ksc3-1841668.pdf" H 4700 7050 50  0001 C CNN
-F 4 "Tactile Switches 0.3mA 24VAC, 1.60N 3.5mmH, J lead, IP67" H 4700 6850 50  0001 C CNN "Description"
-F 5 "C&K" H 4700 6850 50  0001 C CNN "Manufacturer_Name"
-F 6 "KSC2TE01JLFS" H 4700 6850 50  0001 C CNN "Manufacturer_Part_Number"
-F 7 "611-KSC2TE01JLFS" H 4700 6850 50  0001 C CNN "Mouser Part Number"
-F 8 "$0.39/10000" H 4700 6850 50  0001 C CNN "Mouser Price/Stock"
+F 2 "Twig:SW_Push_1P1T-MP_NO_Horizontal_TL6340" H 4700 7050 50  0001 C CNN
+F 3 "https://sten-eswitch-13110800-production.s3.amazonaws.com/system/asset/product_line/data_sheet/256/TL6340.pdf" H 4700 7050 50  0001 C CNN
+F 4 "Tactile Switch SPST-NO Side Actuated Surface Mount, Right Angle" H 4700 6850 50  0001 C CNN "Description"
+F 5 "E-Switch" H 4700 6850 50  0001 C CNN "Manufacturer_Name"
+F 6 "TL6340AF160QG" H 4700 6850 50  0001 C CNN "Manufacturer_Part_Number"
+F 7 "" H 4700 6850 50  0001 C CNN "Mouser Part Number"
+F 8 "$0.48/10000" H 4700 6850 50  0001 C CNN "Mouser Price/Stock"
+F 9 "SKTDLHE010" H 4700 6850 50  0001 C CNN "Alt Part Number 3"
+F 10 "EVP-AKE31A" H 4700 6850 50  0001 C CNN "Alternate Part Number 1"
 	1    4700 6850
 	1    0    0    -1

Commit message: added slot, updated led pins, updated buttons, still working on jtag and which IO to use
Signed-off-by: lokimetasmith <lokimail@gmail.com>
Parts:
- J3: value Conn_01x05_Male -> Conn_01x06_Male; footprint Connector_PinSocket_1.00mm:PinSocket_1x06_P1.00mm_Vertical_SMD_Pin1Right -> Connector_PinHeader_1.00mm:PinHeader_1x07_P1.00mm_Vertical_SMD_Pin1Right; symbol temp-sensor-rescue:Conn_01x05_Male-Connector -> Connector_Generic:Conn_01x07
- SW1, SW2: value SW_Push -> SW_Push_Right_Angle
Connections:
- wire segments 245 -> 247
Other:
- note added: "can't use Ixx GPIO lines"
Changed lines of the file:
@@
 Wire Wire Line
 	5050 1000 5050 1050
-Text Notes 6700 5750 2    50   ~ 0
+Text Notes 7550 5900 2    50   ~ 0
 JTAG\n
-Text Label 7400 6000 2    50   ~ 0
+Text Label 6300 5900 2    50   ~ 0
 TMS
-Text Label 7400 6100 2    50   ~ 0
+Text Label 6300 6000 2    50   ~ 0
 TDI
-Text Label 7400 6200 2    50   ~ 0
+Text Label 6300 6100 2    50   ~ 0
 TCK
-Text Label 7400 6300 2    50   ~ 0
+Text Label 6300 6200 2    50   ~ 0
 TDO
 Wire Wire Line
-	7400 6000 6950 6000
-Wire Wire Line
-	7400 6100 6950 6100
-Wire Wire Line
-	7400 6200 6950 6200
-Wire Wire Line
-	7400 6300 6950 6300
+	6300 5900 5850 5900
+Wire Wire Line
+	6300 6100 5850 6100
+Wire Wire Line
+	6300 6000 5850 6000
+Wire Wire Line
+	6300 6200 5850 6200
 $Comp
 L temp-sensor-rescue:+5V-power #PWR027
@@
 Text Notes 8800 1150 0    50   ~ 0
 AHT20 pin compatable but rotated 180
-Text Label 1950 1550 0    50   ~ 0
+Text Label 1200 1600 0    50   ~ 0
 SCL
-Text Label 1950 1450 0    50   ~ 0
+Text Label 1200 1500 0    50   ~ 0
 SDA
 Text Notes 400  -1650 0    50   ~ 0
@@
 L temp-sensor-rescue:GND-power #PWR0101
 U 1 1 60946B45
-P 7350 6400
-F 0 "#PWR0101" H 7350 6150 50  0001 C CNN
-F 1 "GND" H 7355 6227 50  0000 C CNN
-F 2 "" H 7350 6400 50  0001 C CNN
-F 3 "" H 7350 6400 50  0001 C CNN
-	1    7350 6400
-	1    0    0    -1
-$EndComp
-Wire Wire Line
-	7350 6400 6950 6400
+P 5950 6300
+F 0 "#PWR0101" H 5950 6050 50  0001 C CNN
+F 1 "GND" H 5955 6127 50  0000 C CNN
+F 2 "" H 5950 6300 50  0001 C CNN
+F 3 "" H 5950 6300 50  0001 C CNN
+	1    5950 6300
+	0    -1   1    0
+$EndComp
+Wire Wire Line
+	5850 6300 5950 6300
 Text Notes 8800 1050 0    50   ~ 0
 HDC1080
@@
 $EndComp
 $Comp
-L temp-sensor-rescue:Conn_01x05_Male-Connector J3
+L Connector_Generic:Conn_01x07 J3
 U 1 1 608AA734
-P 6750 6200
-F 0 "J3" H 6850 6600 50  0000 C CNN
-F 1 "Conn_01x05_Male" H 6850 6500 50  0000 C CNN
-F 2 "Connector_PinSocket_1.00mm:PinSocket_1x06_P1.00mm_Vertical_SMD_Pin1Right" H 6750 6200 50  0001 C CNN
-F 3 "~" H 6750 6200 50  0001 C CNN
-	1    6750 6200
-	1    0    0    -1
+P 5650 6100
+F 0 "J3" H 5750 6500 50  0000 C CNN
+F 1 "Conn_01x06_Male" H 5750 6400 50  0000 C CNN
+F 2 "Connector_PinHeader_1.00mm:PinHeader_1x07_P1.00mm_Vertical_SMD_Pin1Right" H 5650 6100 50  0001 C CNN
+F 3 "~" H 5650 6100 50  0001 C CNN
+	1    5650 6100
+	-1   0    0    -1
 $EndComp
 $Comp
@@
 P 3550 6850
 F 0 "SW1" H 3550 7135 50  0000 C CNN
-F 1 "SW_Push" H 3550 7044 50  0000 C CNN
+F 1 "SW_Push_Right_Angle" H 3550 7044 50  0000 C CNN
 F 2 "Twig:SW_Push_1P1T-MP_NO_Horizontal_TL6340" H 3550 7050 50  0001 C CNN
 F 3 "https://sten-eswitch-13110800-production.s3.amazonaws.com/system/asset/product_line/data_sheet/256/TL6340.pdf" H 3550 7050 50  0001 C CNN
@@
 P 4700 6850
 F 0 "SW2" H 4700 7135 50  0000 C CNN
-F 1 "SW_Push" H 4700 7044 50  0000 C CNN
+F 1 "SW_Push_Right_Angle" H 4700 7044 50  0000 C CNN
 F 2 "Twig:SW_Push_1P1T-MP_NO_Horizontal_TL6340" H 4700 7050 50  0001 C CNN
 F 3 "https://sten-eswitch-13110800-production.s3.amazonaws.com/system/asset/product_line/data_sheet/256/TL6340.pdf" H 4700 7050 50  0001 C CNN
@@
 Wire Wire Line
 	4450 5650 4850 5650
+Text Notes 850  950  0    50   ~ 0
+can't use Ixx GPIO lines
+Text Label 6300 5800 2    50   ~ 0
+EN
+$Comp
+L temp-sensor-rescue:+3.3V-power #PWR0114
+U 1 1 613FB3C4
+P 6050 6400
+F 0 "#PWR0114" H 6050 6250 50  0001 C CNN
+F 1 "+3.3V" H 6065 6573 50  0000 C CNN
+F 2 "" H 6050 6400 50  0001 C CNN
+F 3 "" H 6050 6400 50  0001 C CNN
+	1    6050 6400
+	0    1    -1   0
+$EndComp
+Wire Wire Line
+	6300 5800 5850 5800
+Wire Wire Line
+	5850 6400 6050 6400
 $EndSCHEMATC

Commit message: updated footprints for switches, adjusted layout and cleaned up traces.
Needs review but should be ready for second spin.

Signed-off-by: lokimetasmith <lokimail@gmail.com>
Parts:
- IC1: footprint ESP32-C3-MINI-1:ESP32C3MINI1 -> Twig:ESP32C3MINI1
Connections:
- net labels added: LED_Blue, LED_Green, LED_Red
Changed lines of the file:
@@
 Text Notes 8800 1150 0    50   ~ 0
 AHT20 pin compatable but rotated 180
-Text Label 1200 1600 0    50   ~ 0
+Text Label 1400 2950 0    50   ~ 0
 SCL
-Text Label 1200 1500 0    50   ~ 0
+Text Label 1750 3150 0    50   ~ 0
 SDA
 Text Notes 400  -1650 0    50   ~ 0
@@
 	8750 4500 8750 4400
 Wire Wire Line
-	8500 4500 8750 4500
-Wire Wire Line
 	8950 4600 8950 4550
 Wire Wire Line
-	8500 4600 8950 4600
-Wire Wire Line
 	8750 4200 8750 4100
 Wire Wire Line
@@
 Wire Wire Line
 	9150 4200 9150 4100
-Wire Wire Line
-	9150 4400 9150 4600
 Text Label 2000 2550 0    50   ~ 0
 io10
@@
 Wire Wire Line
 	7450 1350 7450 1500
-$Comp
-L temp-sensor-rescue:+3.3V-power #PWR0108
-U 1 1 60BCEE9B
-P 5900 1950
-F 0 "#PWR0108" H 5900 1800 50  0001 C CNN
-F 1 "+3.3V" H 5915 2123 50  0000 C CNN
-F 2 "" H 5900 1950 50  0001 C CNN
-F 3 "" H 5900 1950 50  0001 C CNN
-	1    5900 1950
-	1    0    0    -1
-$EndComp
-Wire Wire Line
-	5900 1950 5900 2000
-Wire Wire Line
-	5550 2000 5900 2000
 $Comp
 L temp-sensor-rescue:GND-power #PWR0109
@@
 F 0 "IC1" H 2800 1315 50  0000 C CNN
 F 1 "ESP32-C3-MINI-1" H 2800 1224 50  0000 C CNN
-F 2 "ESP32-C3-MINI-1:ESP32C3MINI1" H 3300 1150 50  0001 L CNN
+F 2 "Twig:ESP32C3MINI1" H 3300 1150 50  0001 L CNN
 F 3 "https://www.espressif.com/sites/default/files/documentation/esp32-c3-mini-1_datasheet_en.pdf" H 3300 1050 50  0001 L CNN
 F 4 "Smallsized module with onboard PCB antenna" H 3300 950 50  0001 L CNN "Description"
@@
 Wire Wire Line
 	1600 2150 2150 2150
-Wire Wire Line
-	1600 2250 2150 2250
 Text Label 1600 2450 0    50   ~ 0
 IO25_pico
@@
 Wire Wire Line
 	1600 2850 2150 2850
-Wire Wire Line
-	1600 2950 2150 2950
 Wire Wire Line
 	1600 3050 2150 3050
@@
 Wire Wire Line
 	5850 6400 6050 6400
+Text Label 8100 4600 0    50   ~ 0
+LED_Green
+Text Label 8150 4500 0    50   ~ 0
+LED_Blue
+Text Label 9150 4650 0    50   ~ 0
+LED_Red
+Wire Wire Line
+	9150 4400 9150 4650
+Wire Wire Line
+	8100 4600 8950 4600
+Wire Wire Line
+	8150 4500 8750 4500
+Wire Wire Line
+	1400 2250 2150 2250
+Wire Wire Line
+	1400 2950 2150 2950
+Wire Wire Line
+	5550 2000 5900 2000
+Wire Wire Line
+	5900 1950 5900 2000
+$Comp
+L temp-sensor-rescue:+3.3V-power #PWR0108
+U 1 1 60BCEE9B
+P 5900 1950
+F 0 "#PWR0108" H 5900 1800 50  0001 C CNN
+F 1 "+3.3V" H 5915 2123 50  0000 C CNN
+F 2 "" H 5900 1950 50  0001 C CNN
+F 3 "" H 5900 1950 50  0001 C CNN
+	1    5900 1950
+	1    0    0    -1
+$EndComp
 $EndSCHEMATC

Commit message: added layout for usb C, lots of little changes to spacing. Still working out how much voltage protection is nessisary for usb-c
Parts:
- added C6: 0.01u, Capacitor_SMD:C_0603_1608Metric, symbol temp-sensor-rescue:C_Small-Device
- added J1: USB_C_Receptacle_USB2.0, Connector_USB:USB_C_Receptacle_HRO_TYPE-C-31-M-12, symbol Connector:USB_C_Receptacle_USB2.0
- added JP1: Jumper_3_Bridged12, Jumper:SolderJumper-3_P1.3mm_Bridged12_RoundedPad1.0x1.5mm, symbol Jumper:Jumper_3_Bridged12
- added R18: 680k, Resistor_SMD:R_0603_1608Metric, symbol temp-sensor-rescue:R_Small_US-Device
- added R19, R20: 5.1k, Resistor_SMD:R_0603_1608Metric, symbol temp-sensor-rescue:R_Small_US-Device
Connections:
- net labels added: CC1, CC2, Shield, TS1, TS2, TS3, TS4, TS5, TS6
- wire segments 247 -> 295
- no-connect marks 16 -> 19
Other:
- moved on the sheet: C2, C4, C8, C9, D2, J2, J3, J5, J6, L2, R1, R14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

Commit message: added fuse and some layout changes
Signed-off-by: lokimetasmith <lokimail@gmail.com>
Parts:
- added F1: 6V 0.5A, symbol Device:Polyfuse_Small
- added R21, R22: 5.1k, Resistor_SMD:R_0603_1608Metric, symbol temp-sensor-rescue:R_Small_US-Device
- J1: Alternate Part Number 1 (none) -> U262-161N-4BVC11; Description (none) -> USB Connectors USB Type C,2.0, Rec, SMT,TH Shell Stakes; Manufacturer_Name (none) -> GCT; Manufacturer_Part_Number (none) -> USB4105-GF-A; Mouser Part Number (none) -> 640-USB4105-GF-A; Mouser Price/Stock (none) -> $0.81
Connections:
- net labels added: V_USB
- wire segments 295 -> 298
- no-connect marks 19 -> 17
Other:
- note added: "Connectors and LED"
- note added: "Power, Reset and Boot"
- moved on the sheet: C2, C3, C4, C5, C8, C9, D1, J2, J3, J5, J6, L1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

Commit message: Mostly all done, with Rev2. need to do final schematic review and logo
Signed-off-by: lokimetasmith <lokimail@gmail.com>
Parts:
- removed R21, R22: 5.1k, Resistor_SMD:R_0603_1608Metric, symbol temp-sensor-rescue:R_Small_US-Device
- F1: footprint (none) -> Fuse:Fuse_0603_1608Metric
- JP1: footprint Jumper:SolderJumper-3_P1.3mm_Bridged12_RoundedPad1.0x1.5mm -> Twig:Jumper_0603_1608Metric
- U5: symbol temp-sensor-rescue:SN65220-Power_Protection -> twig:SN65220-Power_Protection_passthrough
Connections:
- wire segments 298 -> 300
- no-connect marks 17 -> 19
Other:
- moved on the sheet: F1
Changed lines of the file:
@@
 L temp-sensor-rescue:+5V-power #PWR013
 U 1 1 608B4F61
-P 3100 5400
-F 0 "#PWR013" H 3100 5250 50  0001 C CNN
-F 1 "+5V" H 3115 5573 50  0000 C CNN
-F 2 "" H 3100 5400 50  0001 C CNN
-F 3 "" H 3100 5400 50  0001 C CNN
-	1    3100 5400
+P 3000 5300
+F 0 "#PWR013" H 3000 5150 50  0001 C CNN
+F 1 "+5V" H 3015 5473 50  0000 C CNN
+F 2 "" H 3000 5300 50  0001 C CNN
+F 3 "" H 3000 5300 50  0001 C CNN
+	1    3000 5300
 	1    0    0    -1
 $EndComp
@@
 Connection ~ 3250 5400
 Wire Wire Line
-	3250 5400 3350 5400
+	3250 5400 3300 5400
 $Comp
 L temp-sensor-rescue:GND-power #PWR017
@@
 $EndComp
 $Comp
-L temp-sensor-rescue:SN65220-Power_Protection U5
+L twig:SN65220-Power_Protection_passthrough U5
 U 1 1 60C545EF
 P 8950 5800
@@
 Wire Wire Line
 	1600 3350 2150 3350
-Text Label 1600 3550 0    50   ~ 0
+Text Label 2200 3550 2    50   ~ 0
 IO20_pico
-Text Label 1600 3650 0    50   ~ 0
+Text Label 2200 3650 2    50   ~ 0
 IO7_pico
 Text Label 1450 3750 0    50   ~ 0
@@
 TDO
 Wire Wire Line
-	1400 1550 1200 1550
-Wire Wire Line
 	14650 2950 14200 2950
 Wire Wire Line
@@
 Wire Wire Line
 	15050 3750 14850 3750
-Wire Wire Line
-	1400 1450 1200 1450
 Text Label 15050 2600 2    50   ~ 0
 TMS
@@
 Text Label 15300 4450 2    50   ~ 0
 EN
-Text Label 1200 1550 0    50   ~ 0
-CC1
-Text Label 1200 1450 0    50   ~ 0
-CC2
 $Comp
 L temp-sensor-rescue:GND-power #PWR0115
@@
 F 0 "JP1" H 6100 1604 50  0000 C CNN
 F 1 "Jumper_3_Bridged12" H 6100 1513 50  0000 C CNN
-F 2 "Jumper:SolderJumper-3_P1.3mm_Bridged12_RoundedPad1.0x1.5mm" H 6100 1400 50  0001 C CNN
+F 2 "Twig:Jumper_0603_1608Metric" H 6100 1400 50  0001 C CNN
 F 3 "~" H 6100 1400 50  0001 C CNN
 	1    6100 1400
@@
 L Device:Polyfuse_Small F1
 U 1 1 615B4780
-P 2850 5400
-F 0 "F1" V 2645 5400 50  0000 C CNN
-F 1 "6V 0.5A" V 2736 5400 50  0000 C CNN
-F 2 "" H 2900 5200 50  0001 L CNN
-F 3 "https://www.mouser.com/datasheet/2/54/mffsmf-777670.pdf" H 2850 5400 50  0001 C CNN
-F 4 "Resettable Fuses - PPTC 6Volts 40A" H 2850 5400 50  0001 C CNN "Description"
-F 5 "Bourns" H 2850 5400 50  0001 C CNN "Manufacturer_Name"
-F 6 "MF-FSMF025X-2" H 2850 5400 50  0001 C CNN "Manufacturer_Part_Number"
-F 7 "652-MF-FSMF025X-2" H 2850 5400 50  0001 C CNN "Mouser Part Number"
-F 8 "$0.79/2555" H 2850 5400 50  0001 C CNN "Mouser Price/Stock"
-	1    2850 5400
+P 2750 5400
+F 0 "F1" V 2545 5400 50  0000 C CNN
+F 1 "6V 0.5A" V 2636 5400 50  0000 C CNN
+F 2 "Fuse:Fuse_0603_1608Metric" H 2800 5200 50  0001 L CNN
+F 3 "https://www.mouser.com/datasheet/2/54/mffsmf-777670.pdf" H 2750 5400 50  0001 C CNN
+F 4 "Resettable Fuses - PPTC 6Volts 40A" H 2750 5400 50  0001 C CNN "Description"
+F 5 "Bourns" H 2750 5400 50  0001 C CNN "Manufacturer_Name"
+F 6 "MF-FSMF025X-2" H 2750 5400 50  0001 C CNN "Manufacturer_Part_Number"
+F 7 "652-MF-FSMF025X-2" H 2750 5400 50  0001 C CNN "Mouser Part Number"
+F 8 "$0.79/2555" H 2750 5400 50  0001 C CNN "Mouser Price/Stock"
+	1    2750 5400
 	0    1    1    0
 $EndComp
-Text Label 2550 5250 0    50   ~ 0
+Text Label 2450 5250 0    50   ~ 0
 V_USB
 Wire Wire Line
-	2550 5250 2550 5400
-Wire Wire Line
-	2550 5400 2750 5400
-Wire Wire Line
-	2950 5400 3100 5400
+	2450 5250 2450 5400
+Wire Wire Line
+	2450 5400 2650 5400
+Wire Wire Line
+	2850 5400 3000 5400
 Text Label 7850 3500 0    50   ~ 0
 V_USB
@@
 Wire Notes Line
 	2750 2100 2350 2100
-$Comp
-L temp-sensor-rescue:R_Small_US-Device R22
-U 1 1 617C5E7A
-P 1500 1550
-F 0 "R22" H 1568 1596 50  0000 L CNN
-F 1 "5.1k" H 1568 1505 50  0000 L CNN
-F 2 "Resistor_SMD:R_0603_1608Metric" H 1500 1550 50  0001 C CNN
-F 3 "https://www.mouser.com/datasheet/2/447/Yageo_03_18_2021_PYu_RC_Group_51_RoHS_L_11-2199992.pdf" H 1500 1550 50  0001 C CNN
-F 4 "Thick Film Resistors - SMD 15 kOhms 100-200 mW 0603 1%" H 1500 1550 50  0001 C CNN "Description"
-F 5 "Yageo" H 1500 1550 50  0001 C CNN "Manufacturer_Name"
-F 6 "RC0603FR-1315KL" H 1500 1550 50  0001 C CNN "Manufacturer_Part_Number"
-F 7 "603-RC0603FR-1315KL" H 1500 1550 50  0001 C CNN "Mouser Part Number"
-F 8 "$0.10/78000" H 1500 1550 50  0001 C CNN "Mouser Price/Stock"
-	1    1500 1550
-	0    -1   1    0
-$EndComp
-$Comp
-L temp-sensor-rescue:R_Small_US-Device R21
-U 1 1 617C8781
-P 1500 1450
-F 0 "R21" H 1568 1496 50  0000 L CNN
-F 1 "5.1k" H 1568 1405 50  0000 L CNN
-F 2 "Resistor_SMD:R_0603_1608Metric" H 1500 1450 50  0001 C CNN
-F 3 "https://www.mouser.com/datasheet/2/447/Yageo_03_18_2021_PYu_RC_Group_51_RoHS_L_11-2199992.pdf" H 1500 1450 50  0001 C CNN
-F 4 "Thick Film Resistors - SMD 15 kOhms 100-200 mW 0603 1%" H 1500 1450 50  0001 C CNN "Description"
-F 5 "Yageo" H 1500 1450 50  0001 C CNN "Manufacturer_Name"
-F 6 "RC0603FR-1315KL" H 1500 1450 50  0001 C CNN "Manufacturer_Part_Number"
-F 7 "603-RC0603FR-1315KL" H 1500 1450 50  0001 C CNN "Mouser Part Number"
-F 8 "$0.10/78000" H 1500 1450 50  0001 C CNN "Mouser Price/Stock"
-	1    1500 1450
-	0    1    -1   0
-$EndComp
 Wire Wire Line
 	8350 3800 8550 3800
@@
 NoConn ~ 7600 4600
 NoConn ~ 7600 4700
+NoConn ~ 2150 1450
+NoConn ~ 2150 1550
+$Comp
+L power:PWR_FLAG #FLG0102
+U 1 1 6199CCA5
+P 3300 5300
+F 0 "#FLG0102" H 3300 5375 50  0001 C CNN
+F 1 "PWR_FLAG" H 3300 5473 50  0000 C CNN
+F 2 "" H 3300 5300 50  0001 C CNN
+F 3 "~" H 3300 5300 50  0001 C CNN
+	1    3300 5300
+	1    0    0    -1
+$EndComp
+Wire Wire Line
+	3000 5300 3000 5400
+Connection ~ 3000 5400
+Wire Wire Line
+	3000 5400 3100 5400
+Wire Wire Line
+	3300 5300 3300 5400
+Connection ~ 3300 5400
+Wire Wire Line
+	3300 5400 3350 5400
 $EndSCHEMATC

Commit message: reworked the layout to improve impedance, or so I hope.
Signed-off-by: lokimetasmith <lokimail@gmail.com>
Parts:
- C1, C2, C3, C4, C5, C6, C8, C9: symbol temp-sensor-rescue:C_Small-Device -> temp-sensor-rescue:C_Small-Device-temp-sensor-rescue
- D1: symbol temp-sensor-rescue:D_TVS-Device -> temp-sensor-rescue:D_TVS-Device-temp-sensor-rescue
- J4: symbol temp-sensor-rescue:USB_B_Micro-Connector -> twig:temp-sensor-rescue_USB_B_Micro-Connector
- L1: symbol temp-sensor-rescue:L_Core_Ferrite_Small-Device -> temp-sensor-rescue:L_Core_Ferrite_Small-Device-temp-sensor-rescue
- R1, R10, R11, R12, R13, R14, R15, R16, R17, R18, R19, R2, R20, R3, R4, R5, R6, R7, R8, R9: symbol temp-sensor-rescue:R_Small_US-Device -> temp-sensor-rescue:R_Small_US-Device-temp-sensor-rescue
- SW1, SW2: symbol temp-sensor-rescue:SW_Push-Switch -> temp-sensor-rescue:SW_Push-Switch-temp-sensor-rescue
- U2: symbol temp-sensor-rescue:TLV62569DBV-Regulator_Switching -> temp-sensor-rescue:TLV62569DBV-Regulator_Switching-temp-sensor-rescue
- U3: symbol temp-sensor-rescue:BME280-Sensor -> temp-sensor-rescue:BME280-Sensor-temp-sensor-rescue
- U4: symbol temp-sensor-rescue:Si7020-A20-Sensor_Humidity -> temp-sensor-rescue:Si7020-A20-Sensor_Humidity-temp-sensor-rescue

Commit message: updated bom, exported gerbers
Signed-off-by: lokimetasmith <lokimail@gmail.com>
Parts:
- R19, R20: Description Thick Film Resistors - SMD 15 kOhms 100-200 mW 0603 1% -> Thick Film Resistors - SMD 5.1K ohm 1%; Manufacturer_Name Yageo -> Bourns; Manufacturer_Part_Number RC0603FR-1315KL -> CR0603-FX-5101ELF; Mouser Part Number 603-RC0603FR-1315KL -> 652-CR0603FX-5101ELF
- SW1, SW2: Digikey Part Number (none) -> 141-TL6340AF160QGCT-ND
Other:
- note added: "Set the module to UART Download mode by pulling IO0 (pulled up by default) and IO2 (pulled up by\ndefault) low. The chip IOs are pulled down internally by default."
- note removed: "Accelerometer"
- note removed: "Figure out GPIO and which are actually needed"
- note removed: "Figure out boot pulldown resistors"
- note removed: "KXOB25-12X1F-TR\nMONOCRYS SOLAR CELL 24.5MW 690MV"
- note removed: "LIS2DS12"
- note removed: "LTC3109"
- note removed: "M3406-ADJ\nhttps://lcsc.com/product-detail/DC-DC-Converters_M3406_C83224.html"
- note removed: "MC3479"
- note removed: "Prototype USB interface, confirm it works"
- note removed: "Removing Capacitance soil moisture measuring for now"
- note removed: "Set the module to UART Download mode by pulling IO0 (pulled up by default) and IO2 (pulled down by\ndefault) low. The chip IOs are pulled down internally by default."
- note removed: "ToDo:\n\n"
- note removed: "USB Micro B might need to be IP rated"
- note removed: "check out soil moisture sensor circuit\n"
- note removed: "switching power supply\n"
- moved on the sheet: C2, C4, R6, R7, SW1, SW2
